Commit message: making release commit for SRCP2: Sun Jan 17 17:15:09 CST 2021

File: ros_workspace/install/install/share/srcp2_models_final/urdf/rovers/small_basic/small_rover_drive_motors.xacro (robot description, xacro)
@@ -14,10 +14,19 @@
     <xacro:property name="wheel_ki"  value="0.0"/>
     <xacro:property name="wheel_kd"  value="0.0"/>
-    <xacro:property name="max_wheel_command_speed" value="${pi}"/>
+    <!-- <xacro:property name="max_wheel_command_speed" value="${pi}"/> -->
     <!-- steering motor PID and other constants -->
     <xacro:property name="steer_kp"  value="10"/>
     <xacro:property name="steer_ki"  value="1.0"/>
     <xacro:property name="steer_kd"  value="0.5"/>
-    <xacro:macro name="drive_and_steer_motors">
+    <xacro:macro name="drive_and_steer_motors" params="rover_type">
+        <xacro:if value="${rover_type=='small_scout'}">
+            <xacro:property name="max_wheel_command_speed" value="${2*pi}"/>
+        </xacro:if>
+        <xacro:if value="${rover_type=='small_hauler'}">
+            <xacro:property name="max_wheel_command_speed" value="${1.5*pi}"/>
+        </xacro:if>
+        <xacro:if value="${rover_type=='small_excavator'}">
+            <xacro:property name="max_wheel_command_speed" value="${pi}"/>
+        </xacro:if>
         <!-- DRIVE/WHEEL MOTORS -->
         <motor>

File: ros_workspace/install/install/share/srcp2_models_final/urdf/rovers/small_basic/small_rover_sensors.xacro (robot description, xacro)
@@ -106,5 +106,5 @@
         <parent link="${rover_name}_sensor_bar"/>
         <child link="${rover_name}_left_camera_optical"/>
-        <origin xyz="0.2 0.2 0.05" rpy="0 0 0"/>
+        <origin xyz="0.2 0.2 0.05" rpy="-1.57 0 -1.57"/>
     </joint>
     <!-- The Right Camera Optical Link -->
@@ -114,5 +114,5 @@
         <parent link="${rover_name}_sensor_bar"/>
         <child link="${rover_name}_right_camera_optical"/>
-        <origin xyz="0.2 -0.01 0.05" rpy="0 0 0"/>
+        <origin xyz="0.2 -0.01 0.05" rpy="-1.57 0 -1.57"/>
     </joint>
   </xacro:macro>

File: ros_workspace/install/install/share/srcp2_models_final/urdf/rovers/small_excavator/arm.xacro (robot description, xacro)
@@ -375,4 +375,12 @@
             </plugin>
         </gazebo>
+        <!-- This is the plugin used for the excavator scoop topic -->
+        <gazebo>
+            <plugin name="excavator_scoop" filename="libExcavatorScoop.so">
+                <scoop_link_name>${rover_name}_scoop</scoop_link_name>
+                <scoop_topic_name>scoop_info</scoop_topic_name>
+                <scoop_topic_publish_rate>0.5</scoop_topic_publish_rate>
+            </plugin>
+        </gazebo>
     </xacro:macro>
 </robot>
