Commit message: making release commit for SRCP2: Fri Feb  5 15:40:22 CST 2021

File: ros_workspace/install/share/srcp2_models_final/urdf/rovers/small_basic/small_rover_chassis.xacro (robot description, xacro)
@@ -12,5 +12,5 @@
     <xacro:macro name="small_rover_chassis" params="rover_name">
         <xacro:include filename="../common/universal_chassis.xacro"/>
-        <xacro:property name="chassis_collision_x" value="0.7"/>
+        <xacro:property name="chassis_collision_x" value="1.2"/>
         <xacro:property name="chassis_collision_y" value="0.8"/>
         <xacro:property name="chassis_collision_z" value="0.2"/>

File: ros_workspace/install/share/srcp2_models_final/urdf/rovers/small_scout/volatile_sensor.xacro (robot description, xacro)
@@ -27,5 +27,5 @@
                 <xacro:volatile_sensor_mount_origin/>
                 <geometry>
-                    <cylinder radius="0.1" length="0.1"/>
+                    <cylinder radius="0.1" length="0.01"/>
                 </geometry>
             </collision>
@@ -42,9 +42,30 @@
             <inertial>
                 <xacro:volatile_sensor_mount_origin/>
-                <mass value="2.0"/>
+                <mass value="0.001"/>
                 <xacro:cylinder_inertia
-                    m="2.0"
+                    m="0.001"
                     r="0.1"
-                    h="0.1"/>
+                    h="0.01"/>
+            </inertial>
+        </link>
+        <!-- this guard the sensor colllision ther to fix collission qwerk with revolute.-->
+        <link name="$(arg rover_name)_volatile_sensor_guard">
+            <collision name="${rover_name}_volatile_sensor_collision_guard">
+                <origin
+                    xyz="0 0 0.12"
+                    rpy="0 0 0"/>
+                <geometry>
+                    <cylinder radius="0.11" length="0.50"/>
+                </geometry>
+            </collision>
+            <inertial>
+                <origin
+                    xyz="0 0 0"
+                    rpy="0 0 0"/>
+                <mass value="0.001"/>
+                <xacro:cylinder_inertia
+                    m="0.001"
+                    r="0.11"
+                    h="0.50"/>
             </inertial>
         </link>
@@ -52,23 +73,30 @@
         <link name="$(arg rover_name)_volatile_sensor">
             <collision name="$(arg rover_name)_volatile_sensor_collision">
-                <xacro:volatile_sensor_origin/>
+                <origin
+                    xyz="0 0 0"
+                    rpy="0 0 0"/>
                 <geometry>
-                    <cylinder radius="0.025" length="0.01"/>
+                    <cylinder radius="0.1" length="0.01"/>
                 </geometry>
             </collision>
             <inertial>
                 <xacro:volatile_sensor_mount_origin/>
-                <mass value="0.1"/>
+                <mass value="0.001"/>
                 <xacro:cylinder_inertia
-                    m="0.1"
+                    m="0.001"
                     r="0.025"
                     h="0.01"/>
             </inertial>
         </link>
-        <!-- bolt the sensor box to the chassis -->
+        <!-- bolt the sensor _ to the chassis -->
         <joint name="volatile_sensor_mount_joint" type="fixed">
             <origin xyz="0.67 0.0 -0.1" rpy="0 0 0"/>
             <parent link = "$(arg rover_name)_small_chassis" />
             <child  link = "$(arg rover_name)_volatile_sensor_mount"/>
+        </joint>
+        <joint name="volatile_sensor_guard_joint" type="fixed">
+            <origin xyz="0.67 0.0 -0.1" rpy="0 0 0"/>
+            <parent link = "$(arg rover_name)_small_chassis" />
+            <child  link = "$(arg rover_name)_volatile_sensor_guard"/>
         </joint>
         <!-- fix the sensor tip to the sensor body. This is a revolute joint to
@@ -98,5 +126,5 @@
         <gazebo>
             <plugin filename="libVolatileSensor.so" name="VolatileSensorPlugin">
-                <publish_interval>5.0</publish_interval>
+                <publish_interval>0.2</publish_interval>
                 <publish_inrange_only>false</publish_inrange_only>
                 <sensor_topic>volatile_sensor</sensor_topic>

Commit message: making release commit for SRCP2: Thu Feb 25 16:00:09 CST 2021

File: ros_workspace/install/share/srcp2_models_final/urdf/rovers/small_basic/small_rover_chassis.xacro (robot description, xacro)
@@ -13,5 +13,5 @@
         <xacro:include filename="../common/universal_chassis.xacro"/>
         <xacro:property name="chassis_collision_x" value="1.2"/>
-        <xacro:property name="chassis_collision_y" value="0.8"/>
+        <xacro:property name="chassis_collision_y" value="0.75"/>
         <xacro:property name="chassis_collision_z" value="0.2"/>
         <xacro:universal_chassis

File: ros_workspace/install/share/srcp2_models_final/urdf/rovers/small_basic/small_rover_power.xacro (robot description, xacro)
@@ -35,3 +35,13 @@
             offset_xyz  = "-0.15 0.4 0.2"/>
     </xacro:macro>
+    <gazebo>
+        <plugin name="system_monitor" filename="libSystemMonitorPlugin.so">
+            <startup_power_save>false</startup_power_save>
+            <startup_percent_level>98.0</startup_percent_level>
+            <threshold_percent_emg>10.0</threshold_percent_emg>
+            <threshold_percent_low>25.0</threshold_percent_low>
+            <repair_heal_range>10.0</repair_heal_range>
+            <repair_model_name>repair_station</repair_model_name>
+        </plugin>
+    </gazebo>
 </robot>

File: ros_workspace/install/share/srcp2_models_final/urdf/rovers/small_excavator/arm.xacro (robot description, xacro)
@@ -382,5 +382,5 @@
                 <scoop_link_name>${rover_name}_scoop</scoop_link_name>
                 <scoop_topic_name>scoop_info</scoop_topic_name>
-                <scoop_topic_publish_rate>0.5</scoop_topic_publish_rate>
+                <scoop_topic_publish_rate>5.0</scoop_topic_publish_rate>
             </plugin>
         </gazebo>

File: ros_workspace/install/share/srcp2_models_final/urdf/rovers/small_excavator/small_excavator.xacro (robot description, xacro)
@@ -54,5 +54,5 @@
                     spawning_zone_joint
             </jointName>
-            <updateRate>15</updateRate>
+            <updateRate>100</updateRate>
             <alwaysOn>true</alwaysOn>
         </plugin>

File: ros_workspace/install/share/srcp2_models_final/urdf/rovers/small_hauler/small_hauler.xacro (robot description, xacro)
@@ -50,5 +50,5 @@
                     bin_joint
             </jointName>
-            <updateRate>15</updateRate>
+            <updateRate>100</updateRate>
             <alwaysOn>true</alwaysOn>
         </plugin>

File: ros_workspace/install/share/srcp2_models_final/urdf/rovers/small_scout/small_scout.xacro (robot description, xacro)
@@ -52,5 +52,5 @@
                     volatile_sensor_joint
             </jointName>
-            <updateRate>15</updateRate>
+            <updateRate>100</updateRate>
             <alwaysOn>true</alwaysOn>
         </plugin>
