Commit message: making release commit for SRCP2: Mon Mar 22 13:36:35 CDT 2021

File: ros_workspace/install/share/srcp2_models_final/urdf/rovers/small_basic/small_rover_sensor_motors.xacro (robot description, xacro)
@@ -11,11 +11,11 @@
 <robot xmlns:xacro="http://www.ros.org/wiki/xacro">
     <!-- YAW motor PID and other constants -->
-    <xacro:property name="sensor_pan_kp"  value="5.0"/>
-    <xacro:property name="sensor_pan_ki"  value="1.0"/>
-    <xacro:property name="sensor_pan_kd"  value="0.1"/>
+    <xacro:property name="sensor_pan_kp"  value="150.0"/>
+    <xacro:property name="sensor_pan_ki"  value="0.1"/>
+    <xacro:property name="sensor_pan_kd"  value="0.0"/>
     <!-- PITCH motor PID and other constants -->
-    <xacro:property name="sensor_tilt_kp"  value="5.0"/>
-    <xacro:property name="sensor_tilt_ki"  value="1.0"/>
-    <xacro:property name="sensor_tilt_kd"  value="0.1"/>
+    <xacro:property name="sensor_tilt_kp"  value="150.0"/>
+    <xacro:property name="sensor_tilt_ki"  value="0.1"/>
+    <xacro:property name="sensor_tilt_kd"  value="0.0"/>
     <xacro:macro name="sensor_motors">
         <!-- SENSOR YAW MOTOR -->
@@ -25,7 +25,7 @@
             <ros_topic>sensor/yaw/command/position</ros_topic>
             <start>0</start>
-            <kp>${wheel_kp}</kp>
-            <ki>${wheel_ki}</ki>
-            <kd>${wheel_kd}</kd>
+            <kp>${sensor_pan_kp}</kp>
+            <ki>${sensor_pan_ki}</ki>
+            <kd>${sensor_pan_kd}</kd>
         </motor>
         <!-- SENSOR PITCH MOTOR -->
@@ -35,7 +35,7 @@
             <ros_topic>sensor/pitch/command/position</ros_topic>
             <start>0</start>
-            <kp>${wheel_kp}</kp>
-            <ki>${wheel_ki}</ki>
-            <kd>${wheel_kd}</kd>
+            <kp>${sensor_tilt_kp}</kp>
+            <ki>${sensor_tilt_ki}</ki>
+            <kd>${sensor_tilt_kd}</kd>
         </motor>
     </xacro:macro>

File: ros_workspace/install/share/srcp2_models_final/urdf/rovers/small_basic/small_rover_sensors.xacro (robot description, xacro)
@@ -48,5 +48,5 @@
               lower    = "-${pi}"
               effort   = "10"
-              velocity = "1.0"/>
+              velocity = "0.01"/>
       <!-- Some joint damping is necessary for this joint, as it's a powerful -->
       <!-- motor and a light link. Without this, the PID controller must be  -->
@@ -74,4 +74,5 @@
       </visual>
       <inertial>
+        <origin xyz="0 0.07 0.05" rpy="0 0 0"/>
         <!-- <xacro:sensor_bar pitch_joint_origin/> -->
         <mass value="${camera_mass}"/>
@@ -92,11 +93,11 @@
               lower    = "-${pi/3}"
               effort   = "10"
-              velocity = "1.0"/>
+              velocity = "0.01"/>
      <!-- Some joint damping is necessary for this joint, as it's a powerful -->
      <!-- motor and a light link. Without this, the PID controller must be  -->
      <!-- perfectly tuned to prevent oscillations -->
       <dynamics
-          damping  = "1"
-          friction = "0.5"/>
+          damping  = "10"
+          friction = "1"/>
     </joint>
     <!-- The Left Camera Optical Link -->
