Commit message: making release commit for SRCP2: Fri Mar  5 16:33:40 CST 2021

File: ros_workspace/install/share/srcp2_models_final/urdf/landers/processing/processing_plant.xacro (robot description, xacro)
@@ -13,5 +13,6 @@
     <xacro:arg name="len" 		default="5.40"/>
     <xacro:arg name="rad" 		default="1.801"/>
-    <xacro:arg name="zoffset"	default="0.50"/>
+    <xacro:arg name="zoffset"	default="0.60"/>
+    <xacro:arg name="zoffset_collision"	default="1.60"/>
     <!-- Main Link  -->
     <link name="$(arg name)_link">
@@ -26,6 +27,6 @@
         </inertial>
         <collision>
-            <origin xyz="0 0 1.60"
-                    rpy="0 0 0"/>
+            <origin xyz="0 0 $(arg zoffset_collision)"
+                    rpy="0 0 -${pi/2}"/>
             <geometry>
                 <cylinder
@@ -36,5 +37,5 @@
         <visual>
             <origin xyz="0 0 $(arg zoffset)"
-                    rpy="0 0 0"/>
+                    rpy="0 0 -${pi/2}"/>
             <geometry>
                 <mesh

File: ros_workspace/install/share/srcp2_models_final/urdf/landers/repair/repair_station.xacro (robot description, xacro)
@@ -13,5 +13,6 @@
     <xacro:arg name="len" 		default="4.30"/>
     <xacro:arg name="rad" 		default="3.194"/>
-    <xacro:arg name="zoffset"	default="2.68"/> <!-- Close to Half Len-->
+    <xacro:arg name="zoffset"	default="3.10"/>
+    <xacro:arg name="zoffset_collision"	default="2.05"/>
     <!-- Main Link  -->
     <link name="$(arg name)_link">
@@ -26,5 +27,5 @@
         </inertial>
         <collision>
-            <origin xyz="0 0 1.6"
+            <origin xyz="0 0 $(arg zoffset_collision)"
                     rpy="0 0 0"/>
             <geometry>
@@ -39,5 +40,5 @@
             <geometry>
                 <mesh
-                    filename = "package://srcp2_models_final/meshes/landers/repair/RepairAndRecharge.dae"
+                    filename = "package://srcp2_models_final/meshes/landers/repair/repair-and-recharge3.dae"
                     scale    = "1 1 1"/>
             </geometry>

Commit message: making release commit for SRCP2: Wed Mar 17 16:11:54 CDT 2021

File: ros_workspace/install/share/srcp2_models_final/urdf/landers/processing/processing_plant.xacro (robot description, xacro)
@@ -65,5 +65,5 @@
     <link name="$(arg name)_hopper_zone_link">
         <collision>
-            <origin xyz="0.0 -2.9 0.75" rpy="0.475 0 0"/>
+            <origin xyz="0.0 -2.9 1.25" rpy="0.475 0 0"/>
             <geometry>
                 <box size="2.8 2.0 0.6"/>
@@ -81,5 +81,5 @@
         <parent  link="$(arg name)_link"/>
         <child link="$(arg name)_hopper_zone_link"/>
-        <origin xyz="0 0 $(arg zoffset)" rpy="0 0 0"/>
+        <origin xyz="0 0 0" rpy="0 0 0"/>
         <axis   xyz="0 0 1"/>
     </joint>

File: ros_workspace/install/share/srcp2_models_final/urdf/rovers/small_excavator/arm.xacro (robot description, xacro)
@@ -368,11 +368,9 @@
                 <heightmap_name>heightmap</heightmap_name>
                 <heightmap_collision_name>collision_heightmap</heightmap_collision_name>
-                <digging_heightmap_name>digging_heightmap</digging_heightmap_name>
-                <digging_heightmap_collision_name>collision_digging_heightmap</digging_heightmap_collision_name>
                 <clod_radius>0.05</clod_radius>
                 <max_capacity>5</max_capacity>
                 <max_volatile_radius>2.0</max_volatile_radius>
-                <min_volatile_depth>5.0</min_volatile_depth>
-                <max_volatile_depth>20.0</max_volatile_depth>
+                <initial_volatile_depth>5.0</initial_volatile_depth>
+                <depleted_volatile_depth>25.0</depleted_volatile_depth>
             </plugin>
         </gazebo>

File: ros_workspace/install/share/srcp2_models_final/urdf/rovers/small_excavator/small_excavator.xacro (robot description, xacro)
@@ -18,13 +18,12 @@
     <xacro:include filename="arm.xacro"/>
     <!-- excavator hardware -->
-    <xacro:small_rover_chassis rover_name="$(arg rover_name)"/>
-    <xacro:small_rover_drive rover_name="$(arg rover_name)"/>
-    <!-- <xacro:small_rover_power rover_name="$(arg rover_name)" rover_type="small_excavator"/> -->
-    <xacro:arm chassis_name="$(arg rover_name)_small_chassis" rover_name="$(arg rover_name)"/>
+    <xacro:small_rover_chassis  rover_name="$(arg rover_name)"/>
+    <xacro:small_rover_drive    rover_name="$(arg rover_name)"/>
+    <xacro:arm                  rover_name="$(arg rover_name)" chassis_name="$(arg rover_name)_small_chassis" />
     <!-- standard sensor package -->
     <xacro:include filename="../small_basic/small_rover_sensors.xacro"/>
-    <xacro:small_rover_camera_sensor rover_name="$(arg rover_name)"/>
-    <xacro:small_rover_imu_sensor rover_name="$(arg rover_name)"/>
-    <xacro:small_rover_lidar_sensor rover_name="$(arg rover_name)"/>
+    <xacro:small_rover_camera_sensor    rover_name="$(arg rover_name)"/>
+    <xacro:small_rover_imu_sensor       rover_name="$(arg rover_name)"/>
+    <xacro:small_rover_lidar_sensor     rover_name="$(arg rover_name)"/>
     <xacro:include filename="../small_basic/small_rover_sensors.gazebo"/>
     <!-- includes: motors (drive, sensor and arm) -->

File: ros_workspace/install/share/srcp2_models_final/urdf/rovers/small_hauler/small_hauler.xacro (robot description, xacro)
@@ -18,13 +18,12 @@
     <xacro:include filename="bin.xacro"/>
     <!-- hauler hardware -->
-    <xacro:small_rover_chassis rover_name="$(arg rover_name)"/>
-    <xacro:small_hauler_bin    rover_name="$(arg rover_name)" parent="$(arg rover_name)_small_chassis"/>
-    <xacro:small_rover_drive rover_name="$(arg rover_name)"/>
-    <!-- <xacro:small_rover_power rover_name="$(arg rover_name)" rover_type="small_hauler"/> -->
+    <xacro:small_rover_chassis  rover_name="$(arg rover_name)"/>
+    <xacro:small_rover_drive    rover_name="$(arg rover_name)"/>
+    <xacro:small_hauler_bin     rover_name="$(arg rover_name)" parent="$(arg rover_name)_small_chassis"/>
     <!-- includes: sensors electronics -->
     <xacro:include filename="../small_basic/small_rover_sensors.xacro"/>
-    <xacro:small_rover_camera_sensor rover_name="$(arg rover_name)"/>
-    <xacro:small_rover_imu_sensor rover_name="$(arg rover_name)"/>
-    <xacro:small_rover_lidar_sensor rover_name="$(arg rover_name)"/>
+    <xacro:small_rover_camera_sensor    rover_name="$(arg rover_name)"/>
+    <xacro:small_rover_imu_sensor       rover_name="$(arg rover_name)"/>
+    <xacro:small_rover_lidar_sensor     rover_name="$(arg rover_name)"/>
     <xacro:include filename="../small_basic/small_rover_sensors.gazebo"/>
     <!-- includes: motors (drive, sensor and bin) -->

File: ros_workspace/install/share/srcp2_models_final/urdf/rovers/small_scout/small_scout.xacro (robot description, xacro)
@@ -17,13 +17,11 @@
     <xacro:include filename="../small_basic/small_rover_power.xacro"/>
     <!-- scout hardware -->
-    <xacro:small_rover_chassis rover_name="$(arg rover_name)"/>
-    <xacro:small_rover_drive rover_name="$(arg rover_name)"/>
-    <!-- <xacro:small_rover_power rover_name="$(arg rover_name)" rover_type="small_scout"/> -->
+    <xacro:small_rover_chassis  rover_name="$(arg rover_name)"/>
+    <xacro:small_rover_drive    rover_name="$(arg rover_name)"/>
     <!-- includes: sensor electronics -->
     <xacro:include filename="../small_basic/small_rover_sensors.xacro"/>
-    <xacro:small_rover_camera_sensor rover_name="$(arg rover_name)"/>
-    <xacro:small_rover_imu_sensor rover_name="$(arg rover_name)"/>
-    <xacro:small_rover_lidar_sensor rover_name="$(arg rover_name)"/>
-    <!-- <xacro:volatile_sensor chassis_link="$(arg rover_name)_small_chassis"/> -->
+    <xacro:small_rover_camera_sensor    rover_name="$(arg rover_name)"/>
+    <xacro:small_rover_imu_sensor       rover_name="$(arg rover_name)"/>
+    <xacro:small_rover_lidar_sensor     rover_name="$(arg rover_name)"/>
     <xacro:include filename="../small_basic/small_rover_sensors.gazebo"/>
     <!-- includes: volatile sensor -->

File: ros_workspace/install/share/srcp2_models_final/urdf/rovers/small_scout/volatile_sensor.xacro (robot description, xacro)
@@ -130,6 +130,6 @@
                 <sensor_topic>volatile_sensor</sensor_topic>
                 <sensing_range>2.0</sensing_range>
-                <min_volatile_depth>5.0</min_volatile_depth>
-                <max_volatile_depth>20.0</max_volatile_depth>
+                <initial_volatile_depth>5.0</initial_volatile_depth>
+                <depleted_volatile_depth>25.0</depleted_volatile_depth>
                 <sensor_link>$(arg rover_name)_volatile_sensor</sensor_link>
             </plugin>
