Commit message: making release commit for SRCP2: Mon Mar 29 16:12:32 CDT 2021

File: ros_workspace/install/share/srcp2_models_final/urdf/rovers/small_excavator/arm.xacro (robot description, xacro)
@@ -38,4 +38,6 @@
         <xacro:property name="shoulder_yaw_damping"        value="2.0" />  <!-- Nm/rad/sec -->
         <xacro:property name="shoulder_yaw_friction"       value="1.0" />  <!-- Nm/rad -->
+        <xacro:property name="shoulder_yaw_upper_limit" value="${pi}" />  <!-- rad -->
+        <xacro:property name="shoulder_yaw_lower_limit" value="${-pi}" /> <!-- rad -->
         <xacro:property name="shoulder_pitch_velocity_limit" value="0.5" />       <!-- rad/sec -->
         <xacro:property name="shoulder_pitch_effort_limit"   value="500" />       <!-- Nm -->
@@ -51,5 +53,5 @@
         <xacro:property name="elbow_pitch_lower_limit"    value="${-pi/4}"/>      <!-- rad -->
         <xacro:property name="wrist_pitch_velocity_limit" value="0.5" />       <!-- rad/sec -->
-        <xacro:property name="wrist_pitch_effort_limit"   value="500" />       <!-- Nm -->
+        <xacro:property name="wrist_pitch_effort_limit"   value="15" />       <!-- Nm -->
         <xacro:property name="wrist_pitch_damping"        value="2.0" />       <!-- Nm/rad/sec -->
         <xacro:property name="wrist_pitch_friction"       value="1.0" />       <!-- Nm/rad -->
@@ -115,5 +117,5 @@
 		</link>
 		<!-- Shoulder Yaw Joint -->
-		<joint name="shoulder_yaw_joint" type="continuous">
+		<joint name="shoulder_yaw_joint" type="revolute">
 			<parent link = "${rover_name}_arm_mount"/>
 			<child  link = "${rover_name}_shoulder"/>
@@ -124,5 +126,7 @@
 			<limit
 				effort   = "${shoulder_yaw_effort_limit}"
-				velocity = "${shoulder_yaw_velocity_limit}" />
+				velocity = "${shoulder_yaw_velocity_limit}"
+                lower    = "${shoulder_yaw_lower_limit}"
+				upper    = "${shoulder_yaw_upper_limit}"/>
 			<dynamics
 				damping  = "${shoulder_yaw_damping}"
@@ -241,11 +245,11 @@
             </visual>
             <inertial>
-				<origin xyz="0.02 0.05 0" rpy="0 ${pi} ${pi/2.0}"/>
+				<origin xyz="0.231837 0.05 -0.1012" rpy="0 0 0"/>
                 <mass value = "0.25"/>
-                <xacro:box_inertia
+                 <xacro:box_inertia
                     m = "0.25"
                     x = "0.33"
-                    y = "0.25"
-                    z = "0.15" />
+                    y = "0.40"
+                    z = "0.05" />
             </inertial>
         </link>
